File: pcb/Adafruit/Feather.kicad_pcb (KiCad board)
At the start: 2 copper layers, 51.3 x 23.4 mm, 27 parts, among them J1 Conn_01x02, J2 Conn_01x02, U1 LM4132xMF-3.3, U2 MCP3x62/ST, U3 NCP163ASN330T1G

Commit message: update pcbs
Routing:
- net +5V: track 20.2 -> 16.3 mm, vias 1 -> 2
- net /SS: track 19.9 -> 21.3 mm
- added copper zone on F.Cu, net +5V
Changed lines of the file:
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@@
   (paper "A4")
   (title_block
-    (title "Adafruit MCP3x62R Breakout")
+    (title "Adafruit Feather MCP3x62R Breakout")
     (date "2023-10-10")
     (company "Stefan Herold")
@@
   )
   (layers
-    (0 "F.Cu" signal)
-    (31 "B.Cu" signal)
+    (0 "F.Cu" mixed)
+    (31 "B.Cu" mixed)
     (32 "B.Adhes" user "B.Adhesive")
     (33 "F.Adhes" user "F.Adhesive")
@@
   (segment (start 142.24 78.486) (end 142.24 72.644) (width 0.4) (layer "F.Cu") (net 3))
   (segment (start 142.24 72.644) (end 143.002 71.882) (width 0.4) (layer "F.Cu") (net 3))
-  (segment (start 132.588 65.024) (end 133.541 65.024) (width 0.4) (layer "F.Cu") (net 4))
   (segment (start 133.35 67.31) (end 133.35 66.561) (width 0.4) (layer "F.Cu") (net 4))
-  (segment (start 133.541 65.595) (end 133.35 65.786) (width 0.4) (layer "F.Cu") (net 4))
   (segment (start 133.538 69.408) (end 133.538 68.4585) (width 0.4) (layer "F.Cu") (net 4))
   (segment (start 131.638 68.4585) (end 131.638 69.408) (width 0.4) (layer "F.Cu") (net 4))
@@
   (segment (start 131.638 69.408) (end 131.826 69.596) (width 0.4) (layer "F.Cu") (net 4))
   (segment (start 133.35 66.535) (end 133.363 66.548) (width 0.4) (layer "F.Cu") (net 4))
-  (segment (start 133.35 65.786) (end 133.35 66.535) (width 0.4) (layer "F.Cu") (net 4))
-  (segment (start 133.541 65.024) (end 133.541 65.595) (width 0.4) (layer "F.Cu") (net 4))
   (segment (start 131.826 69.596) (end 133.35 69.596) (width 0.4) (layer "F.Cu") (net 4))
   (segment (start 133.35 69.596) (end 133.538 69.408) (width 0.4) (layer "F.Cu") (net 4))
   (segment (start 133.35 66.561) (end 133.363 66.548) (width 0.4) (layer "F.Cu") (net 4))
-  (via (at 132.588 65.024) (size 0.4) (drill 0.2) (layers "F.Cu" "B.Cu") (net 4))
-  (segment (start 132.588 64.516) (end 133.604 63.5) (width 0.4) (layer "B.Cu") (net 4))
+  (via (at 132.9944 63.5) (size 0.4) (drill 0.2) (layers "F.Cu" "B.Cu") (net 4))
+  (via (at 133.8834 63.5) (size 0.4) (drill 0.2) (layers "F.Cu" "B.Cu") (net 4))
+  (segment (start 132.9944 63.5) (end 141.986 63.5) (width 0.4) (layer "B.Cu") (net 4))
+  (segment (start 142.24 63.246) (end 142.24 62.23) (width 0.4) (layer "B.Cu") (net 4))
   (segment (start 141.986 63.5) (end 142.24 63.246) (width 0.4) (layer "B.Cu") (net 4))
-  (segment (start 142.24 63.246) (end 142.24 62.23) (width 0.4) (layer "B.Cu") (net 4))
-  (segment (start 133.604 63.5) (end 141.986 63.5) (width 0.4) (layer "B.Cu") (net 4))
-  (segment (start 132.588 65.024) (end 132.588 64.516) (width 0.4) (layer "B.Cu") (net 4))
   (via (at 149.352 76.962) (size 0.4) (drill 0.2) (layers "F.Cu" "B.Cu") (net 13))
   (via (at 150.114 74.676) (size 0.4) (drill 0.2) (layers "F.Cu" "B.Cu") (net 13))
@@
   (segment (start 143.663 77.317) (end 144.8485 77.317) (width 0.25) (layer "F.Cu") (net 16))
   (via (at 143.6624 77.3176) (size 0.4) (drill 0.2) (layers "F.Cu" "B.Cu") (net 16))
-  (segment (start 143.6624 77.3176) (end 152.4 68.58) (width 0.25) (layer "B.Cu") (net 16))
-  (segment (start 152.4 68.58) (end 152.4 62.23) (width 0.25) (layer "B.Cu") (net 16))
+  (segment (start 152.4 68.58) (end 146.5834 74.3966) (width 0.25) (layer "B.Cu") (net 16))
+  (segment (start 146.5834 74.3966) (end 144.145 74.3966) (width 0.25) (layer "B.Cu") (net 16))
+  (segment (start 144.145 74.3966) (end 143.6624 74.8792) (width 0.25) (layer "B.Cu") (net 16))
+  (segment (start 143.6624 74.8792) (end 143.6624 77.3176) (width 0.25) (layer "B.Cu") (net 16))
+  (segment (start 152.4 62.23) (end 152.4 68.58) (width 0.25) (layer "B.Cu") (net 16))
   (segment (start 154.94 81.026) (end 154.94 82.55) (width 0.25) (layer "F.Cu") (net 17))
   (segment (start 149.931 76.017) (end 154.94 81.026) (width 0.25) (layer "F.Cu") (net 17))
@@
       )
     )
+  )
+  (zone (net 4) (net_name "+5V") (layer "F.Cu") (hatch edge 0.5)
+    (priority 2)
+    (connect_pads (clearance 0.254))
+    (min_thickness 0.25) (filled_areas_thickness no)
+    (fill yes (thermal_gap 0.5) (thermal_bridge_width 0.5))
+    (polygon
+      (pts
+        (xy 132.5372 62.992)
+        (xy 134.1628 62.992)
+        (xy 134.1628 65.6844)
+        (xy 133.9088 66.04)
+        (xy 133.9088 67.1068)
+        (xy 132.842 67.1068)
+        (xy 132.842 66.04)
+        (xy 132.5372 65.7352)
+        (xy 132.5372 63.5508)
+      )
+    )
