File: pcb/Adafruit/Feather.kicad_sch (KiCad schematic)
At the start: 27 parts, among them J1 Conn_01x02, J2 Conn_01x02, U1 LM4132xMF-3.0, U2 MCP3x62/ST, U3 NCP163ASN330T1G

Commit message: update pcbs
Parts:
- U2: symbol MCP3x6x:MCP3x62/ST -> MCP3x6x:MCP3x62/ST
Other:
- title: Adafruit MCP3x6xR Breakout  -> Adafruit Feather MCP3x6xR Breakout 
Changed lines of the file:
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@@
   (paper "A4")
   (title_block
-    (title "Adafruit MCP3x6xR Breakout ")
+    (title "Adafruit Feather MCP3x6xR Breakout ")
     (date "2023-10-10")
     (rev "0.1")
@@
     (effects (font (size 1.27 1.27)) (justify left bottom))
   )
-  (symbol (lib_id "MCP3x6x:MCP3x62{slash}ST") (at 177.8 127 0) (unit 1)
+  (symbol (lib_id "MCP3x6x:MCP3x62/ST") (at 177.8 127 0) (unit 1)
     (in_bom yes) (on_board yes) (dnp no) (fields_autoplaced)
     (property "Reference" "U2" (at 182.3594 100.33 0)
