File: pcb/Arduino/Uno.kicad_pcb (KiCad board)
At the start: 2 copper layers, 68.6 x 53.3 mm, 34 parts, among them J1 Conn_01x09, U1 LM4132xMF-3.3, U2 MCP3x64/ST, U3 NCP163ASN330T1G

Commit message: update pcbs
Routing:
- net GNDA: vias 50 -> 51
Changed lines of the file:
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@@
   (paper "A4")
   (title_block
-    (title "Arduino MCP3x6xR Breakout")
+    (title "Arduino Uno MCP3x6xR Breakout")
     (date "2023-10-10")
     (company "Stefan Herold")
@@
     (property "Sheetname" "")
     (attr smd)
-    (fp_text reference "R3" (at 0 -1.778 90) (layer "F.SilkS")
+    (fp_text reference "R3" (at -0.002 -1.143 180) (layer "F.SilkS")
         (effects (font (size 1 1) (thickness 0.15)))
     )
@@
     (property "Sheetname" "")
     (attr smd)
-    (fp_text reference "C9" (at 0 -1.16 90) (layer "F.SilkS")
-        (effects (font (size 1 1) (thickness 0.15)))
-    )
-    (fp_text value "10p" (at 0 1.16 90) (layer "F.Fab")
+    (fp_text reference "C9" (at 0 -1.268 90) (layer "F.SilkS")
+        (effects (font (size 1 1) (thickness 0.15)))
+    )
+    (fp_text value "10p" (at 0 1.145 90) (layer "F.Fab")
         (effects (font (size 1 1) (thickness 0.15)))
     )
@@
     (property "Sheetname" "")
     (attr smd)
-    (fp_text reference "C5" (at 0 -1.16 90) (layer "F.SilkS")
+    (fp_text reference "C5" (at 0 -1.268 90) (layer "F.SilkS")
         (effects (font (size 1 1) (thickness 0.15)))
     )
@@
     (property "Sheetname" "")
     (attr smd)
-    (fp_text reference "R8" (at -0.002 -1.778 90) (layer "F.SilkS")
+    (fp_text reference "R8" (at -0.002 -1.143 180) (layer "F.SilkS")
         (effects (font (size 1 1) (thickness 0.15)))
     )
@@
     (property "Sheetname" "")
     (attr smd)
-    (fp_text reference "R10" (at 0 -1.43 90) (layer "F.SilkS")
+    (fp_text reference "R10" (at 0 -1.524 90) (layer "F.SilkS")
         (effects (font (size 1 1) (thickness 0.15)))
     )
@@
         (effects (font (size 1 1) (thickness 0.15)))
     )
-    (fp_text value "1n" (at 0 1.43 90) (layer "F.Fab")
+    (fp_text value "1n" (at -1.143 -3.429 90) (layer "F.Fab")
         (effects (font (size 1 1) (thickness 0.15)))
     )
@@
         (effects (font (size 1 1) (thickness 0.15)))
     )
-    (fp_text value "MCP3x64/ST" (at 0 4.2 90) (layer "F.Fab")
+    (fp_text value "MCP3x64/ST" (at 0 5.842 90) (layer "F.Fab")
         (effects (font (size 1 1) (thickness 0.15)))
     )
@@
         (effects (font (size 1 1) (thickness 0.15)))
     )
-    (fp_text value "100n" (at 0 1.43 90) (layer "F.Fab")
+    (fp_text value "100n" (at -1.143 3.175 90) (layer "F.Fab")
         (effects (font (size 1 1) (thickness 0.15)))
     )
@@
     (property "Sheetname" "")
     (attr smd)
-    (fp_text reference "C10" (at 0 -1.16 90) (layer "F.SilkS")
-        (effects (font (size 1 1) (thickness 0.15)))
-    )
-    (fp_text value "10p" (at 0 1.16 90) (layer "F.Fab")
+    (fp_text reference "C10" (at 0 -1.268 90) (layer "F.SilkS")
+        (effects (font (size 1 1) (thickness 0.15)))
+    )
+    (fp_text value "10p" (at 0 1.145 90) (layer "F.Fab")
         (effects (font (size 1 1) (thickness 0.15)))
     )
@@
     (property "Sheetname" "")
     (attr smd)
-    (fp_text reference "C7" (at 0 -1.16 90) (layer "F.SilkS")
+    (fp_text reference "C7" (at 0 -1.268 90) (layer "F.SilkS")
         (effects (font (size 1 1) (thickness 0.15)))
     )
@@
     (property "Sheetname" "")
     (attr smd)
-    (fp_text reference "R2" (at 0 -1.778 90) (layer "F.SilkS")
+    (fp_text reference "R2" (at -0.002 -1.143 180) (layer "F.SilkS")
         (effects (font (size 1 1) (thickness 0.15)))
     )
@@
     (property "Sheetname" "")
     (attr smd)
-    (fp_text reference "R1" (at 0 -1.778 90) (layer "F.SilkS")
+    (fp_text reference "R1" (at 0 -1.143 180) (layer "F.SilkS")
         (effects (font (size 1 1) (thickness 0.15)))
     )
@@
     (property "Sheetname" "")
     (attr smd)
-    (fp_text reference "R7" (at 0 -1.778 90) (layer "F.SilkS")
+    (fp_text reference "R7" (at -0.002 -1.143 180) (layer "F.SilkS")
         (effects (font (size 1 1) (thickness 0.15)))
     )
@@
     (property "Sheetname" "")
     (attr smd)
-    (fp_text reference "C3" (at 0 -1.16 90) (layer "F.SilkS")
+    (fp_text reference "C3" (at 0 -1.268 90) (layer "F.SilkS")
         (effects (font (size 1 1) (thickness 0.15)))
     )
@@
         (effects (font (size 1 1) (thickness 0.15)))
     )
-    (fp_text value "Arduino_Leonardo" (at 0 22.86) (layer "F.Fab")
-        (effects (font (size 1 1) (thickness 0.15)))
-    )
-    (fp_text user "${REFERENCE}" (at 0 20.32 180) (layer "F.Fab")
+    (fp_text value "Arduino_Leonardo" (at 6.604 7.62) (layer "F.Fab")
+        (effects (font (size 1 1) (thickness 0.15)))
+    )
+    (fp_text user "${REFERENCE}" (at 6.731 5.969 180) (layer "F.Fab")
         (effects (font (size 1 1) (thickness 0.15)))
     )
@@
         (effects (font (size 1 1) (thickness 0.15)))
     )
-    (fp_text value "1n" (at 0 1.43) (layer "F.Fab")
+    (fp_text value "1n" (at 0 -1.397) (layer "F.Fab")
         (effects (font (size 1 1) (thickness 0.15)))
     )
@@
     (property "Sheetname" "")
     (attr smd)
-    (fp_text reference "R4" (at -0.002 -1.778 90) (layer "F.SilkS")
+    (fp_text reference "R4" (at -0.002 -1.143 180) (layer "F.SilkS")
         (effects (font (size 1 1) (thickness 0.15)))
     )
@@
     (property "Sheetname" "")
     (attr through_hole)
-    (fp_text reference "J1" (at 20.32 -6.96 90) (layer "F.SilkS")
+    (fp_text reference "J1" (at -4.318 0 -180) (layer "F.SilkS")
         (effects (font (size 1 1) (thickness 0.15)))
     )
@@
     (property "Sheetname" "")
     (attr smd)
-    (fp_text reference "C6" (at 0 -1.16 90) (layer "F.SilkS")
+    (fp_text reference "C6" (at 0 -1.268 90) (layer "F.SilkS")
         (effects (font (size 1 1) (thickness 0.15)))
     )
@@
     (property "Sheetname" "")
     (attr smd)
-    (fp_text reference "C4" (at 0 -1.16 90) (layer "F.SilkS")
+    (fp_text reference "C4" (at 0 -1.268 90) (layer "F.SilkS")
         (effects (font (size 1 1) (thickness 0.15)))
     )
@@
     (property "Sheetname" "")
     (attr smd)
-    (fp_text reference "R6" (at -0.002 -1.778 90) (layer "F.SilkS")
+    (fp_text reference "R6" (at -0.002 -1.143 180) (layer "F.SilkS")
         (effects (font (size 1 1) (thickness 0.15)))
     )
@@
         (effects (font (size 1 1) (thickness 0.15)))
     )
-    (fp_text value "SolderJumper_3_Open" (at 0 1.9) (layer "F.Fab")
+    (fp_text value "SolderJumper_3_Open" (at 0 1.9) (layer "F.Fab") hide
         (effects (font (size 1 1) (thickness 0.15)))
     )
@@
         (effects (font (size 1 1) (thickness 0.15)))
     )
-    (fp_text value "SolderJumper_3_Open" (at 0 1.9) (layer "F.Fab")
+    (fp_text value "SolderJumper_3_Open" (at 0 1.9) (layer "F.Fab") hide
         (effects (font (size 1 1) (thickness 0.15)))
     )
@@
         (effects (font (size 1 1) (thickness 0.15)))
     )
-    (fp_text value "NCP163ASN330T1G" (at 0 2.4 90) (layer "F.Fab")
+    (fp_text value "NCP163ASN330T1G" (at 0 -5.842 90) (layer "F.Fab")
         (effects (font (size 1 1) (thickness 0.15)))
     )
@@
         (effects (font (size 1 1) (thickness 0.15)))
     )
-    (fp_text value "LM4132xMF-3.3" (at 0 2.4 -270) (layer "F.Fab")
+    (fp_text value "LM4132xMF-3.3" (at 0 3.683 -270) (layer "F.Fab")
         (effects (font (size 1 1) (thickness 0.15)))
     )
@@
         (effects (font (size 1 1) (thickness 0.15)))
     )
-    (fp_text value "100n" (at 0 1.43 90) (layer "F.Fab")
+    (fp_text value "100n" (at -1.778 -3.175 90) (layer "F.Fab")
         (effects (font (size 1 1) (thickness 0.15)))
     )
@@
     (property "Sheetname" "")
     (attr smd)
-    (fp_text reference "C8" (at 0 -1.16 90) (layer "F.SilkS")
+    (fp_text reference "C8" (at 0 -1.268 90) (layer "F.SilkS")
         (effects (font (size 1 1) (thickness 0.15)))
     )
@@
     (property "Sheetname" "")
     (attr smd)
-    (fp_text reference "R5" (at 0 -1.778 90) (layer "F.SilkS")
+    (fp_text reference "R5" (at -0.002 -1.143 180) (layer "F.SilkS")
         (effects (font (size 1 1) (thickness 0.15)))
     )
@@
         (effects (font (size 1 1) (thickness 0.15)))
     )
-    (fp_text value "1n" (at 0 1.43 90) (layer "F.Fab")
+    (fp_text value "1n" (at -1.524 3.429 90) (layer "F.Fab")
         (effects (font (size 1 1) (thickness 0.15)))
     )
@@
   (via (at 140.97 116.332) (size 0.4) (drill 0.2) (layers "F.Cu" "B.Cu") (free) (net 32))
   (via (at 129.286 121.92) (size 0.4) (drill 0.2) (layers "F.Cu" "B.Cu") (free) (net 32))
+  (via (at 128.905 124.841) (size 0.4) (drill 0.2) (layers "F.Cu" "B.Cu") (free) (net 32))
   (via (at 137.16 113.03) (size 0.4) (drill 0.2) (layers "F.Cu" "B.Cu") (free) (net 32))
   (via (at 116.332 111.76) (size 0.4) (drill 0.2) (layers "F.Cu" "B.Cu") (free) (net 32))
