File: pcb/Arduino/Uno.kicad_sch (KiCad schematic)
At the start: 34 parts, among them J1 Conn_01x09, U1 LM4132xMF-3.0, U2 MCP3x64/ST, U3 NCP163ASN330T1G

Commit message: update pcbs
Parts:
- U2: symbol MCP3x6x:MCP3x64/ST -> MCP3x6x:MCP3x64/ST
Other:
- title: Arduino MCP3x6x Breakout  -> Arduino Uno MCP3x6x Breakout 
Changed lines of the file:
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@@
   (paper "A4")
   (title_block
-    (title "Arduino MCP3x6x Breakout ")
+    (title "Arduino Uno MCP3x6x Breakout ")
     (date "2022-12-29")
     (rev "0.1")
@@
     )
   )
-  (symbol (lib_id "MCP3x6x:MCP3x64{slash}ST") (at 177.8 127 0) (unit 1)
+  (symbol (lib_id "MCP3x6x:MCP3x64/ST") (at 177.8 127 0) (unit 1)
     (in_bom yes) (on_board yes) (dnp no) (fields_autoplaced)
     (property "Reference" "U2" (at 182.3594 100.33 0)
