File: pcb/Sparkfun/ProMicro.kicad_sch (KiCad schematic)
At the start: 22 parts, among them J1 Conn_01x02, U2 MCP3x61/NC, U3 TLV75533PDRV, U4 MCP1501-30xRW

Commit message: update pcbs
Parts:
- removed J1: Conn_01x02, Connector_Coaxial:U.FL_Molex_MCRF_73412-0110_Vertical, symbol Connector_Generic:Conn_01x02
- removed U2: MCP3x61/NC, Package_DFN_QFN:QFN-20-1EP_3x3mm_P0.4mm_EP1.65x1.65mm_ThermalVias, symbol MCP3x6x:MCP3x61/NC
- added C10, C5, C6, C7, C8, C9: 10p, Capacitor_SMD:C_0402_1005Metric, symbol Device:C
- added J1: Conn_02x05_Odd_Even, Connector_PinSocket_2.54mm:PinSocket_2x05_P2.54mm_Horizontal, symbol Connector_Generic:Conn_02x05_Odd_Even
- added R3, R4, R5, R6, R7, R8: 1k, Resistor_SMD:R_0402_1005Metric, symbol Device:R
- added U1: MCP3x64/NC, Package_DFN_QFN:QFN-20-1EP_3x3mm_P0.4mm_EP1.65x1.65mm_ThermalVias, symbol MCP3x6x:MCP3x64/NC
- A3: footprint Module:Arduino_Nano -> pcb:ProMicro
Connections:
- net +5V: now also A3.24 (RAW); no longer A3.21 (VCC)
- net GNDA: now also C10.1, C5.2, C6.1, C7.2, C8.1, C9.2, J1.10 (Pin_10), U1.1 (VREF-), U1.20 (AGND)
- net GNDD: now also U1.17 (DGND)
- net IRQ: now also U1.15 (~{IRQ}/MDAT)
- net MCLK: now also J1.9 (Pin_9), U1.16 (MCLK)
- net MISO: now also U1.14 (SDO)
- net MOSI: now also U1.13 (SDI)
- net SCK: now also U1.12 (SCK)
- net SS: now also A3.13 (CS/D10), U1.11 (~{CS}); no longer A3.9 (D6/A7)
- net VDD: now also A3.21 (VCC), U1.18 (DVDD)
- net VDDA: now also U1.19 (AVDD)
- net CH0: now reaches R1.1
- net CH0: now also J1.1 (Pin_1)
- net CH1: now reaches R2.1
- net CH1: now also J1.2 (Pin_2)
- net at C4.2, R2.2: now also U1.4 (CH1)
- net VREF+: now reaches C11.1, C2.1, U4.7 (OUT), U4.8 (FB)
- net VREF+: now also U1.2 (VREF+)
- net at C3.1, R1.2: now also U1.3 (CH0)
- new net: C7.1, R5.2, U1.7 (CH4)
- new net: C5.1, R3.2, U1.5 (CH2)
- new net: C10.2, R8.2, U1.10 (CH7)
- new net: C6.2, R4.2, U1.6 (CH3)
- new net: C8.2, R6.2, U1.8 (CH5)
- new net: C9.1, R7.2, U1.9 (CH6)
- new net CH2: J1.3 (Pin_3), R3.1
- new net CH3: J1.4 (Pin_4), R4.1
- new net CH4: J1.5 (Pin_5), R5.1
- new net CH5: J1.6 (Pin_6), R6.1
- new net CH6: J1.7 (Pin_7), R7.1
- new net CH7: J1.8 (Pin_8), R8.1
Other:
- title: Sparkfun MCP3x6xR Breakout  -> Sparkfun ProMicro MCP3x6xR Breakout 
